File: prog328smd/prog328smd.kicad_pcb (KiCad board)
At the start: 2 copper layers, 5 parts, among them J1 Conn_01x08_Female, J2 Conn_01x08_Female, J3 Conn_01x08_Female, J4 Conn_01x08_Female, U1 ATMEGA328P-AU

Commit message: First Commit
Parts:
- removed J4: Conn_01x08_Female, millk:conn8
- added IC1: DS3231, DS3231:SO16W, F.Cu at (128.3, 74.4)
- added R1: R, Resistors_SMD:R_0805_HandSoldering, F.Cu at (112.8, 64.8)
- added R2: R, Resistors_SMD:R_0805_HandSoldering, F.Cu at (116.3, 64.8)
- added R3: R, Resistors_SMD:R_0805_HandSoldering, F.Cu at (119.8, 64.8)
- added R4: R, Resistors_SMD:R_0805_HandSoldering, F.Cu at (106.3, 69.0)
- added R5: R, Resistors_SMD:R_0805_HandSoldering, F.Cu at (131.5, 83.0)
- added SW1: SW_Push, millk:pushbutton_2pin, F.Cu at (111.0, 81.5)
- J1: value Conn_01x08_Female -> Conn_01x06_Female; footprint millk:conn8 -> millk:conn6
- J3: value Conn_01x08_Female -> Conn_01x02_Female; footprint millk:conn8 -> millk:Conn2
- moved J3 56.4 mm to (127.9, 62.9), turned to 0 degrees
- moved U1 28.3 mm to (115.6, 74.2)
- moved J1 28.2 mm to (114.0, 91.1), turned to 0 degrees
- moved J2 15.6 mm to (120.5, 86.3), turned to 0 degrees
Connections:
- J1 pad 1: Net-(J1-Pad1) -> d10
- J1 pad 2: Net-(J1-Pad2) -> d12
- J1 pad 3: Net-(J1-Pad3) -> d13
- J1 pad 4: Net-(J1-Pad4) -> d11
- J1 pad 5: Net-(J1-Pad5) -> gnd
- J1 pad 6: Net-(J1-Pad6) -> vcc
- J2 pad 1: Net-(J2-Pad1) -> busy
- J2 pad 2: Net-(J2-Pad2) -> reset
- J2 pad 3: Net-(J2-Pad3) -> d.c
- J2 pad 4: Net-(J2-Pad4) -> cs
- J2 pad 5: Net-(J2-Pad5) -> d13
- J2 pad 6: Net-(J2-Pad6) -> d11
- J2 pad 7: Net-(J2-Pad7) -> gnd
- J2 pad 8: Net-(J2-Pad8) -> vcc
- J3 pad 1: Net-(J3-Pad1) -> Net-(IC1-Pad14)
- J3 pad 2: Net-(J3-Pad2) -> gnd
- U1 pad 1: Net-(J3-Pad1) -> Net-(R4-Pad2)
- U1 pad 11: Net-(J4-Pad3) -> busy
- U1 pad 12: Net-(J4-Pad4) -> reset
- U1 pad 13: Net-(J4-Pad5) -> d.c
- U1 pad 14: Net-(J4-Pad6) -> cs
- U1 pad 15: Net-(J4-Pad7) -> d11
- U1 pad 16: Net-(J4-Pad8) -> d12
- U1 pad 17: Net-(J2-Pad1) -> d13
- U1 pad 18: Net-(J2-Pad2) -> vcc
- U1 pad 19: Net-(J2-Pad3) -> Net-(U1-Pad19)
- U1 pad 2: Net-(J3-Pad2) -> rtcVcc
- U1 pad 20: Net-(J2-Pad4) -> vcc
- U1 pad 21: Net-(J2-Pad5) -> gnd
- U1 pad 22: Net-(J2-Pad6) -> Net-(U1-Pad22)
- U1 pad 23: Net-(J2-Pad7) -> Net-(U1-Pad23)
- U1 pad 24: Net-(J2-Pad8) -> Net-(U1-Pad24)
- U1 pad 25: Net-(J1-Pad1) -> Net-(U1-Pad25)
- U1 pad 26: Net-(J1-Pad2) -> Net-(U1-Pad26)
- U1 pad 27: Net-(J1-Pad3) -> sda
- U1 pad 28: Net-(J1-Pad4) -> scl
- U1 pad 29: Net-(J1-Pad5) -> d10
- U1 pad 3: Net-(J2-Pad5) -> gnd
- U1 pad 30: Net-(J1-Pad6) -> Net-(U1-Pad30)
- U1 pad 31: Net-(J1-Pad7) -> Net-(U1-Pad31)
- U1 pad 32: Net-(J1-Pad8) -> Net-(U1-Pad32)
- U1 pad 4: Net-(J3-Pad4) -> vcc
- U1 pad 5: Net-(J2-Pad5) -> gnd
- U1 pad 6: Net-(J3-Pad4) -> vcc
- U1 pad 7: Net-(J3-Pad7) -> Net-(U1-Pad7)
- U1 pad 8: Net-(J3-Pad8) -> Net-(U1-Pad8)
Routing:
- net vcc: track 0.00 -> 53.6 mm
- net d10: track 0.00 -> 49.4 mm
- net Net-(J2-Pad5): track 38.0 -> 0.00 mm
- net gnd: track 0.00 -> 34.1 mm
- net d11: track 0.00 -> 20.6 mm
- net Net-(J3-Pad4): track 19.5 -> 0.00 mm
- net Net-(R4-Pad2): track 0.00 -> 18.5 mm
- net sda: track 0.00 -> 17.7 mm
- net d13: track 0.00 -> 16.0 mm, vias 0 -> 1
- net scl: track 0.00 -> 15.1 mm
- net Net-(J4-Pad8): track 13.8 -> 0.00 mm
- net Net-(U1-Pad9): track 13.6 -> 0.00 mm
- net Net-(J4-Pad7): track 13.1 -> 0.00 mm
- net Net-(U1-Pad10): track 12.9 -> 0.00 mm
- net Net-(J4-Pad6): track 12.4 -> 0.00 mm
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- added copper zone on F.Cu, net gnd
