File: progds32321/progds32321.kicad_pcb (KiCad board)
At the start: 2 copper layers, 3 parts, among them IC1 DS3231, J1 Conn_01x04_Female, J2 Conn_01x04_Female

Commit message: First Commit
Routing:
- added copper zone on F.Cu, net (none)
Changed lines of the file:
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@@
   (segment (start 95.155 50.5) (end 95.1 50.555) (width 0.4) (layer F.Cu) (net 8))
   (segment (start 99.5 50.5) (end 95.155 50.5) (width 0.4) (layer F.Cu) (net 8))
+  (zone (net 0) (net_name "") (layer F.Cu) (hatch edge 0.508)
+    (connect_pads (clearance 0.7))
+    (min_thickness 0.254)
+    (fill yes (arc_segments 32) (thermal_gap 0.508) (thermal_bridge_width 0.508))
+    (polygon
+      (pts
+        (xy 78 48.5) (xy 78 61.5) (xy 78 62) (xy 102 62) (xy 102 48.5)
+      )
+    )
+  )
 )
